Commit message: 你的提交信息

File: src/simple_meca_car/urdf/waking_robot.xacro (robot description, xacro)
@@ -226,17 +226,17 @@
   </link>
      <!-- camera -->
-  <!-- Hokuyo joint -->
-  <joint name="hokuyo_joint" type="fixed">
+<!-- 正面雷达 joint -->
+<joint name="front_laser_joint" type="fixed">
     <origin xyz="0.125 0.0 0.225" rpy="0 0 0"/>
     <parent link="base_link"/>
     <axis xyz="0 1 0" />
-    <child link="laser_frame"/>
-  </joint>
-  <!-- Hokuyo Laser -->
-  <link name="laser_frame">
+    <child link="front_laser_frame"/>
+</joint>
+<!-- 正面雷达 link -->
+<link name="front_laser_frame">
     <collision>
       <origin xyz="0 0 0" rpy="0 0 0"/>
       <geometry>
-	<box size="0.05 0.05 0.05"/>
+        <box size="0.05 0.05 0.05"/>
       </geometry>
     </collision>
@@ -252,5 +252,96 @@
       <inertia ixx="1e-6" ixy="0" ixz="0" iyy="1e-6" iyz="0" izz="1e-6" />
     </inertial>
-  </link>
+</link>
+<!-- 背面雷达 joint -->
+<joint name="back_laser_joint" type="fixed">
+    <origin xyz="-0.125 0.0 0.225" rpy="0 0 ${PI}"/>
+    <parent link="base_link"/>
+    <axis xyz="0 1 0" />
+    <child link="back_laser_frame"/>
+</joint>
+<!-- 背面雷达 link -->
+<link name="back_laser_frame">
+    <collision>
+      <origin xyz="0 0 0" rpy="0 0 0"/>
+      <geometry>
+        <box size="0.05 0.05 0.05"/>
+      </geometry>
+    </collision>
+    <visual>
+      <origin xyz="0 0 0" rpy="0 0 0"/>
+      <geometry>
+        <mesh filename="package://simple_meca_car/meshes/hokuyo.dae"/>
+      </geometry>
+    </visual>
+    <inertial>
+      <mass value="1e-2" />
+      <origin xyz="0 0 0" rpy="0 0 0"/>
+      <inertia ixx="1e-6" ixy="0" ixz="0" iyy="1e-6" iyz="0" izz="1e-6" />
+    </inertial>
+</link>
+<!-- 正面雷达 gazebo 配置 -->
+<gazebo reference="front_laser_frame">
+    <sensor type="ray" name="front_laser_sensor">
+      <pose>0 0 0 0 0 0</pose>
+      <visualize>false</visualize>
+      <update_rate>40</update_rate>
+      <ray>
+        <scan>
+          <horizontal>
+            <samples>720</samples>
+            <resolution>1</resolution>
+            <min_angle>-3.1415926</min_angle>
+            <max_angle>3.1415926</max_angle>
+          </horizontal>
+        </scan>
+        <range>
+          <min>0.05</min>
+          <max>30.0</max>
+          <resolution>0.01</resolution>
+        </range>
+        <noise>
+          <type>gaussian</type>
+          <mean>0.0</mean>
+          <stddev>0.01</stddev>
+        </noise>
+      </ray>
+      <plugin name="gazebo_ros_front_laser_controller" filename="libgazebo_ros_laser.so">
+        <topicName>scan_front</topicName>
+        <frameName>front_laser_frame</frameName>
+      </plugin>
+    </sensor>
+</gazebo>
+<!-- 背面雷达 gazebo 配置 -->
+<gazebo reference="back_laser_frame">
+    <sensor type="ray" name="back_laser_sensor">
+      <pose>0 0 0 0 0 0</pose>
+      <visualize>false</visualize>
+      <update_rate>40</update_rate>
+      <ray>
+        <scan>
+          <horizontal>
+            <samples>720</samples>
+            <resolution>1</resolution>
+            <min_angle>-3.1415926</min_angle>
+            <max_angle>3.1415926</max_angle>
+          </horizontal>
+        </scan>
+        <range>
+          <min>0.05</min>
+          <max>30.0</max>
+          <resolution>0.01</resolution>
+        </range>
+        <noise>
+          <type>gaussian</type>
+          <mean>0.0</mean>
+          <stddev>0.01</stddev>
+        </noise>
+      </ray>
+      <plugin name="gazebo_ros_back_laser_controller" filename="libgazebo_ros_laser.so">
+        <topicName>scan_back</topicName>
+        <frameName>back_laser_frame</frameName>
+      </plugin>
+    </sensor>
+</gazebo>
    <!-- hokuyo -->
 <!-- gazebo插件设置相关 -->
